Commit message: Added gripper and arm camera

File: robots/rbrobout/rbrobout_plus.urdf.xacro (robot description, xacro)
@@ -13,4 +13,6 @@
   <xacro:include
     filename="$(find robotnik_sensors)/urdf/all_sensors.urdf.xacro" />
+  <xacro:include
+    filename="$(find robotnik_description)/urdf/grippers/suction_gripper/suction_gripper.urdf.xacro" />
   <!-- ARGUMENTS -->
   <xacro:arg
@@ -23,4 +25,7 @@
     name="gazebo_ignition"
     default="false" />
+  <xacro:arg
+    name="world_name"
+    default="demo" />
   <xacro:arg
     name="ur_type"
@@ -56,4 +61,20 @@
       rpy="0 0 0" />
   </xacro:arm_ur>
+  <!-- WRIST CAMERA -->
+  <xacro:sensor_intel_realsense_d435i
+    frame_prefix="$(arg prefix)wrist_rgbd_camera_"
+    parent="$(arg prefix)arm_tool0"
+    node_namespace="$(arg namespace)"
+    node_name="wrist_camera"
+    gazebo_ignition="$(arg gazebo_ignition)">
+    <origin xyz="0.0 -0.1 -0.040" rpy="0 -1.5708 1.5708" />
+  </xacro:sensor_intel_realsense_d435i>
+  <!-- SUCTION GRIPPER -->
+  <xacro:suction_gripper
+    prefix="$(arg prefix)vacuum_"
+    parent="$(arg prefix)arm_tool0"
+    ns="$(arg namespace)">
+    <origin xyz="0 0 0" rpy="0 0 0" />
+  </xacro:suction_gripper>
   <!-- IMU -->
   <xacro:sensor_vectornav
@@ -102,3 +123,13 @@
       rpy="0 0 0" />
   </xacro:sensor_intel_realsense_d435>
+<!-- VACUUM GRIPPER PLUGIN -->
+  <gazebo>
+    <plugin filename="libVacuumGripper.so"
+            name="vacuum_gripper_plugin::VacuumGripper">
+      <suction_link>$(arg prefix)vacuum_link_suction_gripper</suction_link>
+      <contact_topic>/world/$(arg world_name)/model/$(arg namespace)/link/$(arg prefix)vacuum_link_suction_gripper/sensor/$(arg prefix)vacuum_suction_contact_sensor/contact</contact_topic>
+      <cmd_topic>/$(arg namespace)/vacuum_on</cmd_topic>
+      <max_distance>0.15</max_distance>
+    </plugin>
+  </gazebo>
 </robot>
